File: numpad-calculator.kicad_pcb (KiCad board)
At the start: 2 copper layers, 53 parts, among them SW1 SW_Push, U1 ProMicro

Commit message: Basic layout
Parts:
- D1, D10, D11, D12, D13, D14, D15, D16, D17, D18, D19, D2, D20, D21, D22, D23, D24, D3, D4, D5, D6, D7, D8, D9, SW1: moved to B.Cu
- moved MX27 233.0 mm to (192.9, 73.8)
- moved MX21 232.5 mm to (192.9, 64.3)
- moved MX1 217.6 mm to (145.3, 73.8)
- moved MX20 211.1 mm to (192.9, 26.2)
- moved MX19 206.3 mm to (173.8, 73.8)
- moved MX26 202.9 mm to (192.9, 54.8)
- moved D18 197.5 mm to (182.2, 73.8), turned to 270 degrees
- moved MX7 192.7 mm to (135.7, 73.8)
- moved MX25 190.9 mm to (192.9, 35.7)
- moved MX18 188.7 mm to (173.8, 54.8)
- moved MX17 181.1 mm to (173.8, 35.7)
- moved D12 179.2 mm to (163.1, 73.8), turned to 270 degrees
- moved MX22 177.2 mm to (192.9, -31.0)
- moved D17 176.5 mm to (182.2, 54.8), turned to 270 degrees
- moved D24 175.1 mm to (184.5, 64.3), turned to 270 degrees
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Connections:
- MX1 pad 1: Col0 -> Col1
- MX1 pad 2: Net-(D6-Pad2) -> Net-(D12-Pad2)
- MX20 pad 2: Net-(D21-Pad2) -> Net-(D22-Pad2)
- MX21 pad 2: Net-(D23-Pad2) -> Net-(D24-Pad2)
